Commit message: update

File: description/robot.urdf.xacro (robot description, xacro)
@@ -2,3 +2,4 @@
 <robot xmlns:xacro="http://www.ros.org/wiki/xacro"  name="robot">
     <xacro:include filename="robot_core.xacro" />
+    <xacro:include filename="gazebo_control.xacro" />
 </robot>

File: description/robot_core.xacro (robot description, xacro)
@@ -44,4 +44,7 @@
         </xacro:inertial_box>
     </link>
+    <gazebo reference="chassis">
+        <material>Gazebo/White</material>
+    </gazebo>
     <!-- LEFT WHEEL -->
     <joint name="left_wheel_joint" type="continuous">
@@ -67,4 +70,7 @@
         </xacro:inertial_cylinder>
     </link>
+    <gazebo reference="left_wheel">
+        <material>Gazebo/Black</material>
+    </gazebo>
     <!-- RIGHT WHEEL -->
     <joint name="right_wheel_joint" type="continuous">
@@ -90,4 +96,7 @@
         </xacro:inertial_cylinder>
     </link>
+    <gazebo reference="right_wheel">
+        <material>Gazebo/Black</material>
+    </gazebo>
     <!-- CASTER WHEEL 1 -->
     <joint name="caster_wheel_joint_1" type="fixed">
@@ -112,4 +121,9 @@
         </xacro:inertial_sphere>
     </link>
+    <gazebo reference="caster_wheel_1">
+        <material>Gazebo/Gray</material>
+        <mu1 value="0.001"/>
+        <mu2 value="0.001"/>
+    </gazebo>
     <!-- CASTER WHEEL 2 -->
     <joint name="caster_wheel_joint_2" type="fixed">
@@ -134,4 +148,9 @@
         </xacro:inertial_sphere>
     </link>
+    <gazebo reference="caster_wheel_2">
+        <material>Gazebo/Gray</material>
+        <mu1 value="0.001"/>
+        <mu2 value="0.001"/>
+    </gazebo>
     <!-- CASTER WHEEL 3 -->
     <joint name="caster_wheel_joint_3" type="fixed">
@@ -156,4 +175,9 @@
         </xacro:inertial_sphere>
     </link>
+    <gazebo reference="caster_wheel_3">
+        <material>Gazebo/Gray</material>
+        <mu1 value="0.001"/>
+        <mu2 value="0.001"/>
+    </gazebo>
     <!-- CASTER WHEEL 4 -->
     <joint name="caster_wheel_joint_4" type="fixed">
@@ -178,3 +202,8 @@
         </xacro:inertial_sphere>
     </link>
+    <gazebo reference="caster_wheel_4">
+        <material>Gazebo/Gray</material>
+        <mu1 value="0.001"/>
+        <mu2 value="0.001"/>
+    </gazebo>
 </robot>

Commit message: update

File: description/robot.urdf.xacro (robot description, xacro)
@@ -1,5 +1,13 @@
 <?xml version="1.0"?>
 <robot xmlns:xacro="http://www.ros.org/wiki/xacro"  name="robot">
+    <xacro:arg name="use_ros2_control" default="true"/>
     <xacro:include filename="robot_core.xacro" />
-    <xacro:include filename="gazebo_control.xacro" />
+    <xacro:if value="$(arg use_ros2_control)">
+        <xacro:include filename="ros2_control.xacro" />
+    </xacro:if>
+    <xacro:unless value="$(arg use_ros2_control)">
+        <xacro:include filename="gazebo_control.xacro" />
+    </xacro:unless>
+    <xacro:include filename="depth_camera.xacro" />
+    <xacro:include filename="lidar.xacro" />
 </robot>

File: description/robot_core.xacro (robot description, xacro)
@@ -34,4 +34,11 @@
             <material name="white"/>
         </visual>
+        <visual>
+            <origin xyz="0.225 0 0.8"/>
+            <geometry>
+                <cylinder radius="0.08" length="1.5"/>
+            </geometry>
+            <material name="white"/>
+        </visual>
         <collision>
             <origin xyz="0.225 0 0.05" rpy="0 0 0"/>
@@ -39,4 +46,11 @@
                 <box size="0.45 0.4 0.1"/>
             </geometry>
+        </collision>
+        <collision>
+            <origin xyz="0.225 0 0.8"/>
+            <geometry>
+                <cylinder radius="0.08" length="1.5"/>
+            </geometry>
+            <material name="white"/>
         </collision>
         <xacro:inertial_box mass="12" x="0.45" y="0.4" z="0.1">
@@ -63,5 +77,5 @@
         <collision>
             <geometry>
-                <cylinder length="0.06" radius="0.065" />
+                <sphere radius="0.065" />
             </geometry>
         </collision>
@@ -89,5 +103,5 @@
         <collision>
             <geometry>
-                <cylinder length="0.06" radius="0.065" />
+                <sphere radius="0.065" />
             </geometry>
         </collision>
